Commit message: Revert "Merge branch 'master' into feat/lowpad-tryout"
This reverts commit a2e635046922399442422f6f01eae24057932e3f, reversing
changes made to 7b1e438feb414f29401c3da1552cab4ebbb0bb4b.

File: zed_wrapper/urdf/include/materials.urdf.xacro (robot description, xacro)
@@ -1,5 +1,5 @@
 <?xml version="1.0"?>
 <!--
-// Copyright 2024 Stereolabs
+// Copyright 2022 Stereolabs
 //
 // Licensed under the Apache License, Version 2.0 (the "License");
@@ -37,9 +37,3 @@
         <color rgba="0.25 0.25 0.25 1.0"/>
     </material>
-    <material name="zedxonegs_mat">
-        <color rgba="0.25 0.25 0.25 1.0"/>
-    </material>
-    <material name="zedxone4k_mat">
-        <color rgba="0.25 0.25 0.25 1.0"/>
-    </material>
 </robot>

File: zed_wrapper/urdf/zed_descr.urdf.xacro (robot description, xacro)
@@ -1,5 +1,5 @@
 <?xml version="1.0"?>
 <!--
-// Copyright 2024 Stereolabs
+// Copyright 2022 Stereolabs
 //
 // Licensed under the Apache License, Version 2.0 (the "License");

File: zed_wrapper/urdf/zed_macro.urdf.xacro (robot description, xacro)
@@ -1,5 +1,5 @@
 <?xml version="1.0"?>
 <!--
-// Copyright 2024 Stereolabs
+// Copyright 2022 Stereolabs
 //
 // Licensed under the Apache License, Version 2.0 (the "License");
@@ -32,8 +32,7 @@
       <xacro:property name="screw_offset_z" value="0.0" />
       <xacro:property name="optical_offset_x" value="-0.01" />
-      <xacro:property name="mono" value="false" />
     </xacro:if>
     <xacro:if value="${model == 'zedm'}">
-      <xacro:property name="baseline" value="0.063" />
+      <xacro:property name="baseline" value="0.06" />
       <xacro:property name="height" value="0.0265" />
       <xacro:property name="bottom_slope" value="0.0" />
@@ -41,5 +40,4 @@
       <xacro:property name="screw_offset_z" value="0.0" />
       <xacro:property name="optical_offset_x" value="0.0" />
-      <xacro:property name="mono" value="false" />
     </xacro:if>
     <xacro:if value="${model == 'zed2'}">
@@ -50,5 +48,4 @@
       <xacro:property name="screw_offset_z" value="0.0" />
       <xacro:property name="optical_offset_x" value="-0.01" />
-      <xacro:property name="mono" value="false" />
     </xacro:if>
     <xacro:if value="${model == 'zed2i'}">
@@ -59,5 +56,4 @@
       <xacro:property name="screw_offset_z" value="0.0" />
       <xacro:property name="optical_offset_x" value="-0.01" />
-      <xacro:property name="mono" value="false" />
     </xacro:if>
     <xacro:if value="${model == 'zedx'}">
@@ -68,5 +64,4 @@
       <xacro:property name="screw_offset_z" value="-0.016" />
       <xacro:property name="optical_offset_x" value="-0.01" />
-      <xacro:property name="mono" value="false" />
     </xacro:if>
     <xacro:if value="${model == 'zedxm'}">
@@ -77,5 +72,4 @@
       <xacro:property name="screw_offset_z" value="-0.016" />
       <xacro:property name="optical_offset_x" value="-0.01" />
-      <xacro:property name="mono" value="false" />
     </xacro:if>
     <xacro:if value="${model == 'virtual'}">
@@ -86,23 +80,4 @@
       <xacro:property name="screw_offset_z" value="-0.0155" />
       <xacro:property name="optical_offset_x" value="0.0" />
-      <xacro:property name="mono" value="false" />
-    </xacro:if>
-    <xacro:if value="${model == 'zedxonegs'}">
-      <xacro:property name="baseline" value="0.0" />
-      <xacro:property name="height" value="0.031" />
-      <xacro:property name="bottom_slope" value="0.0" />
-      <xacro:property name="screw_offset_x" value="0.0" />
-      <xacro:property name="screw_offset_z" value="-0.0155" />
-      <xacro:property name="optical_offset_x" value="0.0" />
-      <xacro:property name="mono" value="true" />
-    </xacro:if>
-    <xacro:if value="${model == 'zedxone4k'}">
-      <xacro:property name="baseline" value="0.0" />
-      <xacro:property name="height" value="0.031" />
-      <xacro:property name="bottom_slope" value="0.0" />
-      <xacro:property name="screw_offset_x" value="0.00" />
-      <xacro:property name="screw_offset_z" value="-0.0155" />
-      <xacro:property name="optical_offset_x" value="0.0" />
-      <xacro:property name="mono" value="true" />
     </xacro:if>
     <!-- Camera mounting point (the threaded screw hole in the bottom) -->
@@ -114,5 +89,5 @@
           <origin xyz="${screw_offset_x} 0 ${screw_offset_z}" rpy="0 0 0"/>
           <geometry>
-<mesh filename="file://$(find zed_msgs)/meshes/${model}.stl"/>
+            <mesh filename="package://zed_interfaces/meshes/${model}.stl" />
           </geometry>
           <material name="${model}_mat" />
@@ -121,5 +96,5 @@
           <origin xyz="${screw_offset_x} 0 ${screw_offset_z}" rpy="0 0 0"/>
           <geometry>
-<mesh filename="file://$(find zed_msgs)/meshes/${model}.stl"/>
+            <mesh filename="package://zed_interfaces/meshes/${model}.stl" />
           </geometry>
         </collision>
@@ -131,104 +106,87 @@
       <origin xyz="0 0 ${height/2}" rpy="0 ${bottom_slope} 0" />
     </joint>
-    <xacro:unless value="${mono}">
-      <!-- Left Camera -->
-      <link name="${name}_left_camera_frame">
-        <xacro:if value="${model == 'virtual'}">
-          <visual>
-            <origin xyz="0 0 0" rpy="0 0 0"/>
-            <geometry>
-  <mesh filename="file://$(find zed_msgs)/meshes/${model}.stl"/>
-            </geometry>
-            <material name="${model}_mat" />
-          </visual>
-          <collision>
-            <origin xyz="0 0 0" rpy="0 0 0"/>
-            <geometry>
-  <mesh filename="file://$(find zed_msgs)/meshes/${model}.stl"/>
-            </geometry>
-          </collision>
-        </xacro:if>
-      </link>
-      <joint name="${name}_left_camera_joint" type="fixed">
+    <!-- Left Camera -->
+    <link name="${name}_left_camera_frame">
+      <xacro:if value="${model == 'virtual'}">
+        <visual>
+          <origin xyz="0 0 0" rpy="0 0 0"/>
+          <geometry>
+            <mesh filename="package://zed_interfaces/meshes/${model}.stl" />
+          </geometry>
+          <material name="${model}_mat" />
+        </visual>
+        <collision>
+          <origin xyz="0 0 0" rpy="0 0 0"/>
+          <geometry>
+            <mesh filename="package://zed_interfaces/meshes/${model}.stl" />
+          </geometry>
+        </collision>
+      </xacro:if>
+    </link>
+    <joint name="${name}_left_camera_joint" type="fixed">
+      <parent link="${name}_camera_center"/>
+      <child link="${name}_left_camera_frame"/>
+      <origin xyz="${optical_offset_x} ${baseline/2} 0" rpy="0 0 0" />
+    </joint>
+    <link name="${name}_left_camera_optical_frame"/>
+    <joint name="${name}_left_camera_optical_joint" type="fixed">
+      <origin xyz="0 0 0" rpy="-${M_PI/2} 0.0 -${M_PI/2}"/>
+      <parent link="${name}_left_camera_frame"/>
+      <child link="${name}_left_camera_optical_frame"/>
+    </joint>
+    <!-- Right Camera -->
+    <link name="${name}_right_camera_frame">
+      <xacro:if value="${model == 'virtual'}">
+        <visual>
+          <origin xyz="0 0 0" rpy="0 0 0"/>
+          <geometry>
+            <mesh filename="package://zed_interfaces/meshes/${model}.stl" />
+          </geometry>
+          <material name="${model}_mat" />
+        </visual>
+        <collision>
+          <origin xyz="0 0 0" rpy="0 0 0"/>
+          <geometry>
+            <mesh filename="package://zed_interfaces/meshes/${model}.stl" />
+          </geometry>
+        </collision>
+      </xacro:if>
+    </link>
+    <joint name="${name}_right_camera_joint" type="fixed">
+      <parent link="${name}_camera_center"/>
+      <child link="${name}_right_camera_frame"/>
+      <origin xyz="${optical_offset_x} -${baseline/2} 0" rpy="0 0 0" />
+    </joint>
+    <link name="${name}_right_camera_optical_frame"/>
+    <joint name="${name}_right_camera_optical_joint" type="fixed">
+      <origin xyz="0 0 0" rpy="-${M_PI/2} 0.0 -${M_PI/2}"/>
+      <parent link="${name}_right_camera_frame"/>
+      <child link="${name}_right_camera_optical_frame"/>
+    </joint>
+    <!-- ZED2 Sensors -->
+    <xacro:if value="${model == 'zed2'}">
+      <link name="${name}_mag_link" />
+      <joint name="${name}_mag_joint" type="fixed">
         <parent link="${name}_camera_center"/>
-        <child link="${name}_left_camera_frame"/>
-        <origin xyz="${optical_offset_x} ${baseline/2} 0" rpy="0 0 0" />
-      </joint>
-      <link name="${name}_left_camera_optical_frame"/>
-      <joint name="${name}_left_camera_optical_joint" type="fixed">
-        <origin xyz="0 0 0" rpy="-${M_PI/2} 0.0 -${M_PI/2}"/>
+        <child link="${name}_mag_link"/>
+        <origin xyz="0 0 0" rpy="0 0 0" />
+      </joint>
+      <link name="${name}_baro_link" />
+      <joint name="${name}_baro_joint" type="fixed">
+        <parent link="${name}_camera_center"/>
+        <child link="${name}_baro_link"/>
+        <origin xyz="0 0 0" rpy="0 0 0" />
+      </joint>
+      <link name="${name}_temp_left_link" />
+      <joint name="${name}_temp_left_joint" type="fixed">
         <parent link="${name}_left_camera_frame"/>
-        <child link="${name}_left_camera_optical_frame"/>
-      </joint>
-      <!-- Right Camera -->
-      <link name="${name}_right_camera_frame">
-        <xacro:if value="${model == 'virtual'}">
-          <visual>
-            <origin xyz="0 0 0" rpy="0 0 0"/>
-            <geometry>
-  <mesh filename="file://$(find zed_msgs)/meshes/${model}.stl"/>
-            </geometry>
-            <material name="${model}_mat" />
-          </visual>
-          <collision>
-            <origin xyz="0 0 0" rpy="0 0 0"/>
-            <geometry>
-  <mesh filename="file://$(find zed_msgs)/meshes/${model}.stl"/>
-            </geometry>
-          </collision>
-        </xacro:if>
-      </link>
-      <joint name="${name}_right_camera_joint" type="fixed">
-        <parent link="${name}_camera_center"/>
-        <child link="${name}_right_camera_frame"/>
-        <origin xyz="${optical_offset_x} -${baseline/2} 0" rpy="0 0 0" />
-      </joint>
-      <link name="${name}_right_camera_optical_frame"/>
-      <joint name="${name}_right_camera_optical_joint" type="fixed">
-        <origin xyz="0 0 0" rpy="-${M_PI/2} 0.0 -${M_PI/2}"/>
+        <child link="${name}_temp_left_link"/>
+        <origin xyz="0 0 0" rpy="0 0 0" />
+      </joint>
+      <link name="${name}_temp_right_link" />
+      <joint name="${name}_temp_right_joint" type="fixed">
         <parent link="${name}_right_camera_frame"/>
-        <child link="${name}_right_camera_optical_frame"/>
-      </joint>
-      <!-- ZED2 Sensors -->
-      <xacro:if value="${model == 'zed2'}">
-        <link name="${name}_mag_link" />
-        <joint name="${name}_mag_joint" type="fixed">
-          <parent link="${name}_camera_center"/>
-          <child link="${name}_mag_link"/>
-          <origin xyz="0 0 0" rpy="0 0 0" />
-        </joint>
-        <link name="${name}_baro_link" />
-        <joint name="${name}_baro_joint" type="fixed">
-          <parent link="${name}_camera_center"/>
-          <child link="${name}_baro_link"/>
-          <origin xyz="0 0 0" rpy="0 0 0" />
-        </joint>
-        <link name="${name}_temp_left_link" />
-        <joint name="${name}_temp_left_joint" type="fixed">
-          <parent link="${name}_left_camera_frame"/>
-          <child link="${name}_temp_left_link"/>
-          <origin xyz="0 0 0" rpy="0 0 0" />
-        </joint>
-        <link name="${name}_temp_right_link" />
-        <joint name="${name}_temp_right_joint" type="fixed">
-          <parent link="${name}_right_camera_frame"/>
-          <child link="${name}_temp_right_link"/>
-          <origin xyz="0 0 0" rpy="0 0 0" />
-        </joint>
-      </xacro:if>
-    </xacro:unless>
-    <xacro:if value="${mono}">
-      <!-- Camera -->
-      <link name="${name}_camera_frame" />
-      <joint name="${name}_camera_joint" type="fixed">
-        <parent link="${name}_camera_center"/>
-        <child link="${name}_camera_frame"/>
-        <origin xyz="${optical_offset_x} 0 0" rpy="0 0 0" />
-      </joint>
-      <link name="${name}_camera_optical_frame"/>
-      <joint name="${name}_camera_optical_joint" type="fixed">
-        <origin xyz="0 0 0" rpy="-${M_PI/2} 0.0 -${M_PI/2}"/>
-        <parent link="${name}_camera_frame"/>
-        <child link="${name}_camera_optical_frame"/>
+        <child link="${name}_temp_right_link"/>
+        <origin xyz="0 0 0" rpy="0 0 0" />
       </joint>
     </xacro:if>
